Commit message: feat: upgrade robot camera to RGBD

File: renato_robot/urdf/renato_robot.xacro (robot description, xacro)
@@ -64,172 +64,179 @@
     <parent link="base_chassis"/>
   </joint>
-<link name='sup_chassis'>
-  <inertial>
-    <mass value="3"/>
-    <origin xyz="0 0 0" rpy=" 0 0 0"/>
-    <cuboid_inertia m="3" x= "0.3" y= "0.3" z="0.05"/>
-    <inertia ixx="0.023125" ixy = "0" ixz = "0" iyy="0.023125" iyz = "0" izz="0.045" />
-  </inertial>
-  <collision name='collision'>
-    <origin xyz="0 0 0" rpy=" 0 0 0"/>
-    <geometry>
-      <box size="0.3 0.3 0.05"/>
-    </geometry>
-  </collision>
-  <visual name='chassis_visual'>
-    <origin xyz="0 0 0" rpy=" 0 0 0"/>
-    <geometry>
-      <box size="0.3 0.3 0.05"/>
-    </geometry>
-  </visual>
-  <collision name='caster_collision'>
-    <origin xyz="-0.12 0 -0.025" rpy=" 0 0 0"/>
-    <geometry>
-      <sphere radius="0.029"/>
-    </geometry>
-  </collision>
-  <visual name='caster_visual'>
-    <origin xyz="-0.12 0 -0.025" rpy=" 0 0 0"/>
-    <geometry>
-      <sphere radius="0.03"/>
-    </geometry>
-  </visual>
-</link>
-<joint type="fixed" name="sup_chassis_joint">
-  <origin xyz="-0.25 0 -0.045" rpy="0 0 0"/>
-  <child link="sup_chassis"/>
-  <parent link="base_chassis"/>
-</joint>
-<!-- Add a weigth bar on the end of the robot's bucket - (TEST ONLY) -->
-<link name='back_sup_chassis'>
-  <inertial>
-    <mass value="0.1"/>
-    <origin xyz="0 0 0" rpy=" 0 0 0"/>
-    <inertia ixx="0.0007708" ixy = "0" ixz = "0" iyy="0.000021667" iyz = "0" izz="0.0007508" />
-  </inertial>
-  <collision name='collision'>
-    <origin xyz="0 0 0" rpy=" 0 0 0"/>
-    <geometry>
-      <box size="0.01 0.3 0.05"/>
-    </geometry>
-  </collision>
-  <visual name='back_sup_chassis_visual'>
-    <origin xyz="0 0 0" rpy=" 0 0 0"/>
-    <geometry>
-      <box size="0.01 0.3 0.05"/>
-    </geometry>
-  </visual>
-</link>
-<joint type="fixed" name="back_sup_chassis_joint">
-  <origin xyz="-0.155 0 0" rpy="0 0 0"/>
-  <child link="back_sup_chassis"/>
-  <parent link="sup_chassis"/>
-</joint>
-<!-- ### WHEELS ### -->
-<link name='left_wheel'>
-  <inertial>
-    <mass value="0.5"/>
-    <origin xyz="0.0 0 0" rpy=" 0 1.5707 1.5707"/>
-    <inertia ixx="0.001904" ixy = "0" ixz = "0" iyy="0.001904" iyz = "0" izz="0.0036" />
-  </inertial>
-  <collision name='collision'>
-    <origin xyz="0.0 0 0" rpy=" 0 1.5707 1.5707"/>
-    <geometry>
-      <cylinder radius="0.12" length="0.05" />
-    </geometry>
-  </collision>
-  <visual name='left_wheel_visual'>
-    <origin xyz="0.0 0 0" rpy=" 0 1.5707 1.5707"/>
-    <geometry>
-      <cylinder radius="0.12" length="0.05" />
-    </geometry>
-  </visual>
-</link>
-<link name='right_wheel'>
-  <inertial>
-    <mass value="0.5"/>
-    <origin xyz="0.0 0 0" rpy=" 0 1.5707 1.5707"/>
-    <inertia ixx="0.001904" ixy = "0" ixz = "0" iyy="0.001904" iyz = "0" izz="0.0036" />
-  </inertial>
-  <collision name='collision'>
-    <origin xyz="0.0 0 0" rpy=" 0 1.5707 1.5707"/>
-    <geometry>
-      <cylinder radius="0.12" length="0.05" />
-    </geometry>
-  </collision>
-  <visual name='right_wheel_visual'>
-    <origin xyz="0.0 0 0" rpy=" 0 1.5707 1.5707"/>
-    <geometry>
-      <cylinder radius="0.12" length="0.05" />
-    </geometry>
-  </visual>
-</link>
-<joint type="continuous" name="left_wheel_hinge">
-  <origin xyz="0 0.185 0.02" rpy="0 0 0"/>
-  <child link="left_wheel"/>
-  <parent link="base_chassis"/>
-  <axis xyz="0 1 0" rpy="0 0 0"/>
-  <limit effort="100" velocity="100"/>
-  <dynamics damping="0.1" friction="0.1"/>
-</joint>
-<joint type="continuous" name="right_wheel_hinge">
-  <origin xyz="0 -0.185 0.02" rpy="0 0 0"/>
-  <child link="right_wheel"/>
-  <parent link="base_chassis"/>
-  <axis xyz="0 1 0" rpy="0 0 0"/>
-  <limit effort="100" velocity="100"/>
-  <dynamics damping="0.1" friction="0.1"/>
-</joint>
-<!-- ### CAMERA ### -->
-<link name="camera">
-  <inertial>
-    <mass value="0.1"/>
-    <origin xyz="0.0 0 0" rpy=" 0 0 0"/>
-    <inertia ixx="1e-6" ixy="0" ixz="0" iyy="1e-6" iyz="0" izz="1e-6" />
-  </inertial>
-  <collision name='camera_collision'>
-    <origin xyz="0 0 0" rpy=" 0 0 0"/>
-    <geometry>
-      <box size="0.05 0.05 0.05"/>
-    </geometry>
-  </collision>
-  <visual name='camera_visual'>
-    <origin xyz="0 0 0" rpy=" 0 0 0"/>
-    <geometry>
-      <box size="0.05 0.05 0.05"/>
-    </geometry>
-  </visual>
-</link>
-<joint type="fixed" name="camera_joint">
-  <origin xyz="0.125 0 0" rpy="0 0 0"/>
-  <child link="camera"/>
-  <parent link="base_chassis"/>
-  <axis xyz="0 1 0" rpy="0 0 0.02"/>
-</joint>
-<!-- ### LIDAR ### -->
-<link name="hokuyo">
-  <inertial>
-    <mass value="1e-5"/>
-    <origin xyz="0.0 0 0" rpy=" 0 0 0"/>
-    <inertia ixx="1e-6" ixy="0" ixz="0" iyy="1e-6" iyz="0" izz="1e-6" />
-  </inertial>
-  <collision name='hokuyo_collision'>
-    <origin xyz="0 0 0" rpy=" 0 0 0"/>
-    <geometry>
-      <box size="0.1 0.1 0.1"/>
-    </geometry>
-  </collision>
-  <visual name='hokuyo_visual'>
-    <origin xyz="0 0 0" rpy=" 0 0 0"/>
-    <geometry>
-      <mesh filename="package://renato_robot/meshes/hokuyo.dae"/>
-    </geometry>
-  </visual>
-</link>
-<joint type="fixed" name="hokuyo_joint">
-  <origin xyz="0 0 0.075" rpy="0 0 0"/>
-  <child link="hokuyo"/>
-  <parent link="base_hokuyo"/>
-  <axis xyz="0 1 0" rpy="0 0 0"/>
-</joint>
+  <link name='sup_chassis'>
+    <inertial>
+      <mass value="3"/>
+      <origin xyz="0 0 0" rpy=" 0 0 0"/>
+      <cuboid_inertia m="3" x= "0.3" y= "0.3" z="0.05"/>
+      <inertia ixx="0.023125" ixy = "0" ixz = "0" iyy="0.023125" iyz = "0" izz="0.045" />
+    </inertial>
+    <collision name='collision'>
+      <origin xyz="0 0 0" rpy=" 0 0 0"/>
+      <geometry>
+        <box size="0.3 0.3 0.05"/>
+      </geometry>
+    </collision>
+    <visual name='chassis_visual'>
+      <origin xyz="0 0 0" rpy=" 0 0 0"/>
+      <geometry>
+        <box size="0.3 0.3 0.05"/>
+      </geometry>
+    </visual>
+    <collision name='caster_collision'>
+      <origin xyz="-0.12 0 -0.025" rpy=" 0 0 0"/>
+      <geometry>
+        <sphere radius="0.029"/>
+      </geometry>
+    </collision>
+    <visual name='caster_visual'>
+      <origin xyz="-0.12 0 -0.025" rpy=" 0 0 0"/>
+      <geometry>
+        <sphere radius="0.03"/>
+      </geometry>
+    </visual>
+  </link>
+  <joint type="fixed" name="sup_chassis_joint">
+    <origin xyz="-0.25 0 -0.045" rpy="0 0 0"/>
+    <child link="sup_chassis"/>
+    <parent link="base_chassis"/>
+  </joint>
+  <!-- Add a weigth bar on the end of the robot's bucket - (TEST ONLY) -->
+  <link name='back_sup_chassis'>
+    <inertial>
+      <mass value="0.1"/>
+      <origin xyz="0 0 0" rpy=" 0 0 0"/>
+      <inertia ixx="0.0007708" ixy = "0" ixz = "0" iyy="0.000021667" iyz = "0" izz="0.0007508" />
+    </inertial>
+    <collision name='collision'>
+      <origin xyz="0 0 0" rpy=" 0 0 0"/>
+      <geometry>
+        <box size="0.01 0.3 0.05"/>
+      </geometry>
+    </collision>
+    <visual name='back_sup_chassis_visual'>
+      <origin xyz="0 0 0" rpy=" 0 0 0"/>
+      <geometry>
+        <box size="0.01 0.3 0.05"/>
+      </geometry>
+    </visual>
+  </link>
+  <joint type="fixed" name="back_sup_chassis_joint">
+    <origin xyz="-0.155 0 0" rpy="0 0 0"/>
+    <child link="back_sup_chassis"/>
+    <parent link="sup_chassis"/>
+  </joint>
+  <!-- ### WHEELS ### -->
+  <link name='left_wheel'>
+    <inertial>
+      <mass value="0.5"/>
+      <origin xyz="0.0 0 0" rpy=" 0 1.5707 1.5707"/>
+      <inertia ixx="0.001904" ixy = "0" ixz = "0" iyy="0.001904" iyz = "0" izz="0.0036" />
+    </inertial>
+    <collision name='collision'>
+      <origin xyz="0.0 0 0" rpy=" 0 1.5707 1.5707"/>
+      <geometry>
+        <cylinder radius="0.12" length="0.05" />
+      </geometry>
+    </collision>
+    <visual name='left_wheel_visual'>
+      <origin xyz="0.0 0 0" rpy=" 0 1.5707 1.5707"/>
+      <geometry>
+        <cylinder radius="0.12" length="0.05" />
+      </geometry>
+    </visual>
+  </link>
+  <link name='right_wheel'>
+    <inertial>
+      <mass value="0.5"/>
+      <origin xyz="0.0 0 0" rpy=" 0 1.5707 1.5707"/>
+      <inertia ixx="0.001904" ixy = "0" ixz = "0" iyy="0.001904" iyz = "0" izz="0.0036" />
+    </inertial>
+    <collision name='collision'>
+      <origin xyz="0.0 0 0" rpy=" 0 1.5707 1.5707"/>
+      <geometry>
+        <cylinder radius="0.12" length="0.05" />
+      </geometry>
+    </collision>
+    <visual name='right_wheel_visual'>
+      <origin xyz="0.0 0 0" rpy=" 0 1.5707 1.5707"/>
+      <geometry>
+        <cylinder radius="0.12" length="0.05" />
+      </geometry>
+    </visual>
+  </link>
+  <joint type="continuous" name="left_wheel_hinge">
+    <origin xyz="0 0.185 0.02" rpy="0 0 0"/>
+    <child link="left_wheel"/>
+    <parent link="base_chassis"/>
+    <axis xyz="0 1 0" rpy="0 0 0"/>
+    <limit effort="100" velocity="100"/>
+    <dynamics damping="0.1" friction="0.1"/>
+  </joint>
+  <joint type="continuous" name="right_wheel_hinge">
+    <origin xyz="0 -0.185 0.02" rpy="0 0 0"/>
+    <child link="right_wheel"/>
+    <parent link="base_chassis"/>
+    <axis xyz="0 1 0" rpy="0 0 0"/>
+    <limit effort="100" velocity="100"/>
+    <dynamics damping="0.1" friction="0.1"/>
+  </joint>
+  <!-- ### CAMERA ### -->
+  <link name="camera_link">
+    <inertial>
+      <mass value="0.1"/>
+      <origin xyz="0.0 0 0" rpy=" 0 0 0"/>
+      <inertia ixx="1e-6" ixy="0" ixz="0" iyy="1e-6" iyz="0" izz="1e-6" />
+    </inertial>
+    <collision name='camera_collision'>
+      <origin xyz="0 0 0" rpy=" 0 0 0"/>
+      <geometry>
+        <box size="0.05 0.05 0.05"/>
+      </geometry>
+    </collision>
+    <visual name='camera_visual'>
+      <origin xyz="0 0 0" rpy=" 0 0 0"/>
+      <geometry>
+        <box size="0.05 0.05 0.05"/>
+      </geometry>
+    </visual>
+  </link>
+  <joint type="fixed" name="camera_joint">
+    <origin xyz="0.125 0 0" rpy="0 0 0"/>
+    <child link="camera"/>
+    <parent link="base_chassis"/>
+    <axis xyz="0 1 0" rpy="0 0 0.02"/>
+  </joint>
+  <joint name="camera_optical_joint" type="fixed">
+    <origin xyz="0 0 0" rpy="-1.5707 0 -1.5707"/>
+    <parent link="camera_link"/>
+    <child link="camera_link_optical"/>
+  </joint>
+  <link name="camera_link_optical">
+  </link>
+  <!-- ### LIDAR ### -->
+  <link name="hokuyo">
+    <inertial>
+      <mass value="1e-5"/>
+      <origin xyz="0.0 0 0" rpy=" 0 0 0"/>
+      <inertia ixx="1e-6" ixy="0" ixz="0" iyy="1e-6" iyz="0" izz="1e-6" />
+    </inertial>
+    <collision name='hokuyo_collision'>
+      <origin xyz="0 0 0" rpy=" 0 0 0"/>
+      <geometry>
+        <box size="0.1 0.1 0.1"/>
+      </geometry>
+    </collision>
+    <visual name='hokuyo_visual'>
+      <origin xyz="0 0 0" rpy=" 0 0 0"/>
+      <geometry>
+        <mesh filename="package://renato_robot/meshes/hokuyo.dae"/>
+      </geometry>
+    </visual>
+  </link>
+  <joint type="fixed" name="hokuyo_joint">
+    <origin xyz="0 0 0.075" rpy="0 0 0"/>
+    <child link="hokuyo"/>
+    <parent link="base_hokuyo"/>
+    <axis xyz="0 1 0" rpy="0 0 0"/>
+  </joint>
 </robot>

Commit message: fix: fixed camera_link references

File: renato_robot/urdf/renato_robot.xacro (robot description, xacro)
@@ -203,5 +203,5 @@
   <joint type="fixed" name="camera_joint">
     <origin xyz="0.125 0 0" rpy="0 0 0"/>
-    <child link="camera"/>
+    <child link="camera_link"/>
     <parent link="base_chassis"/>
     <axis xyz="0 1 0" rpy="0 0 0.02"/>

Commit message: fix: Added more features to map and adjust .launch

File: renato_robot/urdf/renato_robot.xacro (robot description, xacro)
@@ -24,6 +24,5 @@
       <mass value="10"/>
       <origin xyz="0 0 0" rpy=" 0 0 0"/>
-      <cuboid_inertia m="10" x= "0.2" y= "0.3" z="0.14"/>
-      <inertia ixx="0.09133" ixy = "0" ixz = "0" iyy="0.04967" iyz = "0" izz="0.0685" />
+      <inertia ixx="0.09133" ixy = "0" ixz = "0" iyy="0.04967" iyz = "0" izz="0.10833" />
     </inertial>
     <collision name='collision'>
@@ -68,5 +67,4 @@
       <mass value="3"/>
       <origin xyz="0 0 0" rpy=" 0 0 0"/>
-      <cuboid_inertia m="3" x= "0.3" y= "0.3" z="0.05"/>
       <inertia ixx="0.023125" ixy = "0" ixz = "0" iyy="0.023125" iyz = "0" izz="0.045" />
     </inertial>
@@ -129,7 +127,7 @@
   <link name='left_wheel'>
     <inertial>
-      <mass value="0.5"/>
-      <origin xyz="0.0 0 0" rpy=" 0 1.5707 1.5707"/>
-      <inertia ixx="0.001904" ixy = "0" ixz = "0" iyy="0.001904" iyz = "0" izz="0.0036" />
+      <mass value="2"/>
+      <origin xyz="0.0 0 0" rpy=" 0 1.5707 1.5707"/>
+      <inertia ixx="0.007617" ixy = "0" ixz = "0" iyy="0.007617" iyz = "0" izz="0.0144" />
     </inertial>
     <collision name='collision'>
@@ -148,7 +146,7 @@
   <link name='right_wheel'>
     <inertial>
-      <mass value="0.5"/>
-      <origin xyz="0.0 0 0" rpy=" 0 1.5707 1.5707"/>
-      <inertia ixx="0.001904" ixy = "0" ixz = "0" iyy="0.001904" iyz = "0" izz="0.0036" />
+      <mass value="2"/>
+      <origin xyz="0.0 0 0" rpy=" 0 1.5707 1.5707"/>
+      <inertia ixx="0.007617" ixy = "0" ixz = "0" iyy="0.007617" iyz = "0" izz="0.0144" />
     </inertial>
     <collision name='collision'>
@@ -171,5 +169,5 @@
     <axis xyz="0 1 0" rpy="0 0 0"/>
     <limit effort="100" velocity="100"/>
-    <dynamics damping="0.1" friction="0.1"/>
+    <dynamics damping="0.01" friction="0.1"/>
   </joint>
   <joint type="continuous" name="right_wheel_hinge">
@@ -179,5 +177,5 @@
     <axis xyz="0 1 0" rpy="0 0 0"/>
     <limit effort="100" velocity="100"/>
-    <dynamics damping="0.1" friction="0.1"/>
+    <dynamics damping="0.01" friction="0.1"/>
   </joint>
   <!-- ### CAMERA ### -->
@@ -202,5 +200,5 @@
   </link>
   <joint type="fixed" name="camera_joint">
-    <origin xyz="0.125 0 0" rpy="0 0 0"/>
+    <origin xyz="0.125 0 0.15" rpy="0 0 0"/>
     <child link="camera_link"/>
     <parent link="base_chassis"/>
